File: eagle/555-dev.brd (EAGLE design)
At the start: 50 x 50 mm, 25 parts, among them IC1 NE555, J3-1 M02PTH, Q1 IRF740, T1 2N2222

Commit message: beta
Parts:
- removed R5: 1K, SparkFun-Resistors:AXIAL-0.4
- removed R7: 220, SparkFun-Resistors:AXIAL-0.4
- added R2: PHOTOCELLPTH-KIT, SparkFun-Sensors:PHOTOCELL-KIT
- C1: value (none) -> 100uF
- R1: value PHOTOCELLPTH-KIT -> 1K; device SparkFun-Sensors:PHOTOCELL-KIT -> SparkFun-Resistors:AXIAL-0.4
- R4: value (none) -> 220
- moved R1 24.9 mm to (32.4, 28.6), turned to 270 degrees
- moved R4 22.9 mm to (9.55, 30.0), turned to 0 degrees
- moved R3 13.0 mm to (25.9, 10.4), turned to 180 degrees
Connections:
- net 555_DISCH: now also R1.P$1, R2.1; no longer R3.P$1
- net 555_TRIG: no longer R1.1, R4.P$2
- net N$11: no longer R4.P$1
- net N$13: no longer R1.2
- net N$7: now also R3.P$1; no longer R5.P$1
- net N$9: now also R4.P$1; no longer R7.P$1
- net OUT: now also R3.P$2, R4.P$2; no longer R5.P$2, R7.P$2
- net VCC: now also R1.P$2, R2.2; no longer R3.P$2
Routing:
- net 555_TRIG: track 33.9 -> 25.6 mm
- net VCC: track 109.1 -> 115.6 mm
- net N$11: track 10.5 -> 4.73 mm
- net N$13: track 10.6 -> 5.24 mm
- net 555_DISCH: track 43.9 -> 48.0 mm
- net OUT: track 68.1 -> 66.2 mm
Other:
- board text added: "+ -"
- board text added: "- +"
- board text added: "Black"
- board text added: "Red"

Commit message: beta
Parts:
- moved D1 5.01 mm to (40.0, 16.2)
- moved D4 2.60 mm to (39.8, 34.5), turned to 90 degrees
Connections:
- net GND: no longer D1.A, D4.A
- net LOAD1-: now also D1.A; no longer D1.C
- net LOAD2-: now also D4.A; no longer D4.C
- net VCC: now also D1.C, D4.C
Routing:
- net VCC: track 115.6 -> 127.9 mm
- net GND: track 10.3 -> 2.70 mm
- net N$1: track 4.73 -> 0.00 mm
- net LOAD2-: track 8.89 -> 11.6 mm
- net LOAD1-: track 9.01 -> 11.4 mm
Changed lines of the file:
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@@
 </element>
 <element name="D3" library="SparkFun-DiscreteSemi" package="DIODE-1N4148-KIT" value="1N4007" x="28.55" y="37.9" smashed="yes" rot="R90">
-<attribute name="NAME" x="31.28" y="34.06" size="1.27" layer="25" font="vector" ratio="10" rot="R90"/>
-<attribute name="VALUE" x="31.258" y="36.868" size="1.27" layer="21" font="vector" ratio="10" rot="R90"/>
+<attribute name="NAME" x="31.08" y="34.06" size="1.27" layer="25" font="vector" ratio="10" rot="R90"/>
+<attribute name="VALUE" x="31.058" y="36.868" size="1.27" layer="21" font="vector" ratio="10" rot="R90"/>
 </element>
 <element name="IC1" library="SUC" package="DIL08" value="NE555" x="18.83" y="21.85" smashed="yes" rot="R180">
@@
 </element>
 <element name="T1" library="adafruit" package="TO92-EBC-OVAL" value="2N2222" x="37.48" y="17.56" smashed="yes" rot="R270">
-<attribute name="NAME" x="40.8" y="21.242" size="1.27" layer="25" font="vector" ratio="10" rot="R180"/>
-<attribute name="VALUE" x="40.8" y="22.892" size="1.27" layer="27" font="vector" ratio="10" rot="R180"/>
+<attribute name="NAME" x="31.058" y="21.2" size="1.27" layer="25" font="vector" ratio="10" rot="R270"/>
+<attribute name="VALUE" x="32.808" y="21.2" size="1.27" layer="27" font="vector" ratio="10" rot="R270"/>
 </element>
 <element name="VR" library="SparkFun-Electromechanical" package="ALPS_POT_KIT" value="50K" x="21.32" y="34.71" smashed="yes" rot="R90">
 <attribute name="PROD_ID" value="RES-09177" x="21.32" y="34.71" size="1.778" layer="27" rot="R90" display="off"/>
-<attribute name="NAME" x="18.58" y="42.89" size="1.27" layer="21" font="vector" ratio="10"/>
-<attribute name="VALUE" x="21.88" y="42.89" size="1.27" layer="21" font="vector" ratio="10"/>
+<attribute name="NAME" x="18.58" y="43.39" size="1.27" layer="21" font="vector" ratio="10"/>
+<attribute name="VALUE" x="21.88" y="43.39" size="1.27" layer="21" font="vector" ratio="10"/>
 </element>
 <element name="J3-1" library="SparkFun-Connectors" package="1X02" value="M02PTH" x="27.5" y="4.6" smashed="yes" rot="R180"/>
 <element name="C1" library="SparkFun-Capacitors" package="CPOL-RADIAL-100UF-25V" value="100uF" x="45.4" y="24.7" smashed="yes">
 <attribute name="VALUE" x="42.495" y="28.182" size="1.27" layer="27" font="vector" ratio="10"/>
-<attribute name="NAME" x="42.538" y="29.651" size="1.27" layer="25" font="vector" ratio="10"/>
+<attribute name="NAME" x="42.538" y="29.851" size="1.27" layer="25" font="vector" ratio="10"/>
 </element>
 <element name="C3" library="SparkFun-Passives" package="CAP-PTH-SMALL" value="0.1uF" x="25.2" y="15.3" smashed="yes" rot="R180">
@@
 <attribute name="VALUE" x="24.546" y="14.224" size="1.27" layer="27" font="vector" ratio="10" rot="R180"/>
 </element>
-<element name="D1" library="SparkFun-DiscreteSemi" package="DIODE-1N4148-KIT" value="1N4007" x="39.7" y="11.2" smashed="yes" rot="R90">
-<attribute name="NAME" x="42.23" y="7.26" size="1.27" layer="25" font="vector" ratio="10" rot="R90"/>
-<attribute name="VALUE" x="38.408" y="7.168" size="1.27" layer="21" font="vector" ratio="10" rot="R90"/>
-</element>
-<element name="D4" library="SparkFun-DiscreteSemi" package="DIODE-1N4148-KIT" value="1N4007" x="39.7" y="37.1" smashed="yes" rot="R270">
-<attribute name="NAME" x="38.23" y="39.16" size="1.27" layer="25" font="vector" ratio="10" rot="R90"/>
-<attribute name="VALUE" x="42.108" y="39.068" size="1.27" layer="21" font="vector" ratio="10" rot="R90"/>
+<element name="D1" library="SparkFun-DiscreteSemi" package="DIODE-1N4148-KIT" value="1N4007" x="40" y="16.2" smashed="yes" rot="R90">
+<attribute name="NAME" x="40.07" y="11.44" size="1.27" layer="25" font="vector" ratio="10" rot="R270"/>
+<attribute name="VALUE" x="38.592" y="11.332" size="1.27" layer="21" font="vector" ratio="10" rot="R270"/>
+</element>
+<element name="D4" library="SparkFun-DiscreteSemi" package="DIODE-1N4148-KIT" value="1N4007" x="39.8" y="34.5" smashed="yes" rot="R90">
+<attribute name="NAME" x="41.03" y="39.46" size="1.27" layer="25" font="vector" ratio="10" rot="R90"/>
+<attribute name="VALUE" x="39.208" y="39.568" size="1.27" layer="21" font="vector" ratio="10" rot="R90"/>
 </element>
 <element name="H5" library="holes" package="3,2" value="MOUNT-HOLE3.2" x="4.1" y="4.1"/>
@@
 <contactref element="C1" pad="2"/>
 <contactref element="C3" pad="1"/>
-<contactref element="D1" pad="A"/>
-<contactref element="D4" pad="A"/>
-<wire x1="39.7" y1="40.91" x2="37.81" y2="40.91" width="0.8128" layer="1"/>
-<wire x1="37.81" y1="40.91" x2="36.2" y2="39.3" width="0.8128" layer="1"/>
-<wire x1="36.2" y1="39.3" x2="36.2" y2="35.96" width="0.8128" layer="1"/>
-<wire x1="36.2" y1="35.96" x2="36.25" y2="35.91" width="0.8128" layer="1"/>
+<wire x1="36.2" y1="35.96" x2="36.25" y2="35.91" width="0" layer="19" extent="1-16"/>
+<wire x1="44.13" y1="24.7" x2="36.25" y2="35.91" width="0" layer="19" extent="1-1"/>
+<wire x1="36.21" y1="20.1" x2="44.13" y2="24.7" width="0" layer="19" extent="1-1"/>
+<wire x1="25.2" y1="15.3" x2="36.21" y2="20.1" width="0" layer="19" extent="1-1"/>
+<wire x1="15.05" y1="12.41" x2="25.2" y2="15.3" width="0" layer="19" extent="1-1"/>
+<wire x1="22.64" y1="25.66" x2="25.2" y2="15.3" width="0" layer="19" extent="1-1"/>
+<wire x1="27.5" y1="4.6" x2="25.2" y2="15.3" width="0" layer="19" extent="1-1"/>
+<wire x1="4.51" y1="23.58" x2="15.05" y2="12.41" width="0" layer="19" extent="1-1"/>
 </signal>
 <signal name="N$5">
@@
 <wire x1="27.6" y1="23.6" x2="32.24" y2="23.6" width="0.8128" layer="1"/>
 <wire x1="32.24" y1="23.6" x2="32.37" y2="23.47" width="0.8128" layer="1"/>
-</signal>
-<signal name="N$11">
-<contactref element="D3" pad="C"/>
-<contactref element="VR" pad="P$1"/>
-<wire x1="23.82" y1="41.71" x2="28.55" y2="41.71" width="0.8128" layer="1"/>
+<contactref element="D1" pad="C"/>
+<contactref element="D4" pad="C"/>
+<wire x1="45.1" y1="36.8" x2="40.054" y2="36.8" width="0.8128" layer="1"/>
+<wire x1="40.054" y1="36.8" x2="39.8" y2="37.054" width="0.8128" layer="1" curve="-90"/>
+<wire x1="39.8" y1="37.054" x2="39.8" y2="38.31" width="0.8128" layer="1"/>
+<wire x1="45" y1="18.5" x2="41.51" y2="18.5" width="0.8128" layer="1"/>
+<wire x1="41.51" y1="18.5" x2="40" y2="20.01" width="0.8128" layer="1"/>
 </signal>
 <signal name="N$13">
@@
 <signal name="LOAD1-">
 <contactref element="T1" pad="C"/>
-<contactref element="D1" pad="C"/>
-<wire x1="39.675859375" y1="15" x2="39.7" y2="15.01" width="0.8128" layer="1" curve="45"/>
-<wire x1="39.86899375" y1="14.94" x2="39.7" y2="15.01" width="0.8128" layer="1" curve="-45"/>
 <contactref element="JP1" pad="2"/>
-<wire x1="45" y1="15" x2="39.71" y2="15" width="0.8128" layer="1"/>
-<wire x1="39.71" y1="15" x2="39.7" y2="15.01" width="0.8128" layer="1"/>
-<wire x1="36.21" y1="15.02" x2="39.69" y2="15.02" width="0.8128" layer="1"/>
-<wire x1="39.69" y1="15.02" x2="39.7" y2="15.01" width="0.8128" layer="1"/>
+<contactref element="D1" pad="A"/>
+<wire x1="36.21" y1="15.02" x2="40" y2="15.02" width="0.8128" layer="1"/>
+<wire x1="40" y1="15.02" x2="45" y2="15.02" width="0.8128" layer="1"/>
+<wire x1="45" y1="15.02" x2="45" y2="15" width="0.8128" layer="1"/>
+<wire x1="40" y1="12.39" x2="40" y2="15.02" width="0.8128" layer="1"/>
 </signal>
 <signal name="LOAD2-">
 <contactref element="Q1" pad="D"/>
-<contactref element="D4" pad="C"/>
-<wire x1="36.25" y1="33.37" x2="39.62" y2="33.37" width="0.8128" layer="1"/>
-<wire x1="39.62" y1="33.37" x2="39.7" y2="33.29" width="0.8128" layer="1"/>
-<wire x1="39.7" y1="33.29" x2="45.09" y2="33.29" width="0.8128" layer="1"/>
 <contactref element="JP2" pad="2"/>
-<wire x1="45.09" y1="33.29" x2="45.1" y2="33.3" width="0.8128" layer="1"/>
+<contactref element="D4" pad="A"/>
+<wire x1="36.25" y1="33.37" x2="39.9" y2="33.37" width="0.8128" layer="1"/>
+<wire x1="39.9" y1="33.37" x2="45.03" y2="33.37" width="0.8128" layer="1"/>
+<wire x1="45.03" y1="33.37" x2="45.1" y2="33.3" width="0.8128" layer="1" curve="-90"/>
+<wire x1="39.8" y1="30.69" x2="39.9" y2="30.79" width="0.8128" layer="1" curve="90"/>
+<wire x1="39.9" y1="30.79" x2="39.9" y2="33.37" width="0.8128" layer="1"/>
+</signal>
+<signal name="N$1">
+<contactref element="D3" pad="C"/>
+<contactref element="VR" pad="P$1"/>
+<wire x1="23.82" y1="41.71" x2="28.55" y2="41.71" width="0" layer="19" extent="1-1"/>
 </signal>
 </signals>
