File: eagle/555-dev.brd (EAGLE design)
At the start: 50 x 50 mm, 25 parts, among them IC1 NE555, Q1 IRF740, T1 2N2222

Commit message: add one more photoresistor and change the R network
user can use the PINS and VR(max/min) to stable the high pulse or the
low one
while the  frequency is modulated by photoresistors, duty cycle changes
due to the static pulse width
simulation: http://goo.gl/erNx82
Layout to be done
Parts:
- added PR2: PHOTOCELLPTH-KIT, SparkFun-Sensors:PHOTOCELL-KIT
- renumbered R2 to PR1
Connections:
- net N$2 renamed PR1
- removed net N$1: D3.C, VR.P$1
- removed net N$13: D2.A, VR.P$3
- new net N$2: D2.C, PR2.1, VR.P$1
- new net N$4: C4.1, D2.A, D3.C
- new net PR2: J1.3, PR2.2
- net 555_DISCH: now also J1.2, VR.P$2; no longer D2.C, D3.A, PR1.1
- net 555_TRIG: no longer C4.1, VR.P$2
- net N$3: now also D3.A, PR1.1, VR.P$3; no longer J1.3, R1.P$2
- net VCC: now also R1.P$2; no longer J1.2
Routing:
- net 555_DISCH: track 47.3 -> 0.00 mm, vias 2 -> 0
- net 555_TRIG: track 25.6 -> 8.75 mm
- net N$3: track 10.2 -> 0.00 mm
- net N$13: track 5.24 -> 0.00 mm
- net VCC: track 121.1 -> 116.5 mm
- net PR1: track 2.70 -> 0.00 mm
Changed lines of the file:
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@@
 <attribute name="PROD_ID" value="CONN-08399" x="45.1" y="36.8" size="1.778" layer="27" rot="R270" display="off"/>
 </element>
-<element name="R2" library="SparkFun-Sensors" package="PHOTOCELL-KIT" value="PHOTOCELLPTH-KIT" x="27.6" y="25.6" smashed="yes" rot="R270">
+<element name="PR1" library="SparkFun-Sensors" package="PHOTOCELL-KIT" value="PHOTOCELLPTH-KIT" x="27.6" y="25.6" smashed="yes" rot="R270">
 <attribute name="NAME" x="27.3" y="22.5" size="1.27" layer="25" font="vector" ratio="10" rot="R270"/>
 </element>
 <element name="J1" library="SparkFun-Connectors" package="1X03" value="" x="27.6" y="20.9" rot="R270"/>
+<element name="PR2" library="SparkFun-Sensors" package="PHOTOCELL-KIT" value="PHOTOCELLPTH-KIT" x="35.6" y="6.4" rot="R270"/>
 </elements>
 <signals>
@@
 <wire x1="45" y1="18.5" x2="41.51" y2="18.5" width="0.8128" layer="1"/>
 <wire x1="41.51" y1="18.5" x2="40" y2="20.01" width="0.8128" layer="1"/>
-<contactref element="J1" pad="2"/>
-<wire x1="27.6" y1="18.36" x2="22.96" y2="18.36" width="0.8128" layer="1"/>
 <wire x1="22.96" y1="18.36" x2="22.64" y2="18.04" width="0.8128" layer="1"/>
-</signal>
-<signal name="N$13">
-<contactref element="D2" pad="A"/>
-<contactref element="VR" pad="P$3"/>
-<wire x1="18.82" y1="41.71" x2="13.81" y2="41.71" width="0.8128" layer="1"/>
-<wire x1="13.81" y1="41.71" x2="13.65" y2="41.55" width="0.8128" layer="1"/>
+<contactref element="R1" pad="P$2"/>
+<wire x1="40" y1="20.01" x2="32.37" y2="23.47" width="0" layer="19" extent="1-1"/>
 </signal>
 <signal name="555_TRIG">
 <contactref element="IC1" pad="2"/>
 <contactref element="IC1" pad="6"/>
-<contactref element="C4" pad="1"/>
-<contactref element="VR" pad="P$2"/>
 <wire x1="20.1" y1="25.66" x2="20.07" y2="25.66" width="0.8128" layer="1"/>
-<wire x1="20.07" y1="25.66" x2="20.07" y2="28.35" width="0.8128" layer="1"/>
-<wire x1="20.07" y1="28.35" x2="20.07" y2="30.17" width="0.8128" layer="1"/>
-<wire x1="20.07" y1="30.17" x2="21.1" y2="31.2" width="0.8128" layer="1"/>
-<wire x1="21.1" y1="31.2" x2="21.1" y2="41.5" width="0.8128" layer="1"/>
-<wire x1="21.1" y1="41.5" x2="21.1" y2="41.79" width="0.8128" layer="1"/>
 <wire x1="20.1" y1="25.66" x2="20.1" y2="23.4" width="0.8128" layer="1"/>
 <wire x1="20.1" y1="23.4" x2="17.5" y2="20.8" width="0.8128" layer="1"/>
 <wire x1="17.5" y1="20.8" x2="17.5" y2="18.1" width="0.8128" layer="1"/>
 <wire x1="17.5" y1="18.1" x2="17.56" y2="18.04" width="0.8128" layer="1"/>
-<wire x1="21.32" y1="41.71" x2="21.31" y2="41.71" width="0.8128" layer="1"/>
-<wire x1="21.31" y1="41.71" x2="21.1" y2="41.5" width="0.8128" layer="1"/>
-</signal>
-<signal name="555_DISCH">
-<contactref element="D3" pad="A"/>
-<contactref element="D2" pad="C"/>
-<contactref element="IC1" pad="7"/>
-<wire x1="13.65" y1="33.93" x2="13.65" y2="37.05" width="0.8128" layer="1"/>
-<wire x1="13.65" y1="37.05" x2="15.3" y2="38.7" width="0.8128" layer="1"/>
-<wire x1="15.3" y1="38.7" x2="19.9" y2="38.7" width="0.8128" layer="1"/>
-<via x="19.9" y="38.7" extent="1-16" drill="0.6" shape="octagon"/>
-<wire x1="19.9" y1="38.7" x2="22.4" y2="38.7" width="0.8128" layer="16"/>
-<via x="22.4" y="38.7" extent="1-16" drill="0.6" shape="octagon"/>
-<wire x1="22.4" y1="38.7" x2="27.1" y2="38.7" width="0.8128" layer="1"/>
-<wire x1="27.1" y1="38.7" x2="28.6" y2="37.2" width="0.8128" layer="1"/>
-<wire x1="28.6" y1="37.2" x2="28.6" y2="34.14" width="0.8128" layer="1"/>
-<wire x1="28.6" y1="34.14" x2="28.55" y2="34.09" width="0.8128" layer="1"/>
-<wire x1="20.1" y1="18.04" x2="20.1" y2="19.794790625" width="0.8128" layer="1"/>
-<wire x1="20.1" y1="19.794790625" x2="20.17439375" y2="19.97439375" width="0.8128" layer="1" curve="-44.999502"/>
-<wire x1="20.17439375" y1="19.97439375" x2="24.6" y2="24.4" width="0.8128" layer="1"/>
-<wire x1="24.6" y1="24.4" x2="24.6" y2="27.194790625" width="0.8128" layer="1"/>
-<wire x1="24.6" y1="27.194790625" x2="24.67439375" y2="27.37439375" width="0.8128" layer="1" curve="-44.999502"/>
-<wire x1="24.67439375" y1="27.37439375" x2="25.6" y2="28.3" width="0.8128" layer="1"/>
-<contactref element="R2" pad="1"/>
-<wire x1="28.55" y1="34.09" x2="28.55" y2="34.05" width="0.8128" layer="1"/>
-<wire x1="25.6" y1="28.3" x2="27.7" y2="28.3" width="0.8128" layer="1"/>
-<wire x1="27.7" y1="28.3" x2="27.7" y2="33.24" width="0.8128" layer="1"/>
-<wire x1="27.7" y1="33.24" x2="28.55" y2="34.09" width="0.8128" layer="1"/>
-<wire x1="28.6" y1="34.14" x2="31.86" y2="34.14" width="0.8128" layer="1"/>
-<wire x1="27.6" y1="27.6" x2="27.7" y2="28.3" width="0.8128" layer="1"/>
-<contactref element="R1" pad="P$1"/>
-<wire x1="31.86" y1="34.14" x2="32.37" y2="33.63" width="0" layer="19" extent="1-1"/>
 </signal>
 <signal name="LOAD1-">
@@
 <wire x1="39.9" y1="30.79" x2="39.9" y2="33.37" width="0.8128" layer="1"/>
 </signal>
-<signal name="N$1">
+<signal name="555_DISCH">
+<contactref element="R1" pad="P$1"/>
+<contactref element="VR" pad="P$2"/>
+<contactref element="IC1" pad="7"/>
+<contactref element="J1" pad="2"/>
+<wire x1="21.32" y1="41.71" x2="32.37" y2="33.63" width="0" layer="19" extent="1-1"/>
+<wire x1="27.6" y1="18.36" x2="32.37" y2="33.63" width="0" layer="19" extent="1-1"/>
+<wire x1="20.1" y1="18.04" x2="27.6" y2="18.36" width="0" layer="19" extent="1-1"/>
+</signal>
+<signal name="N$2">
+<contactref element="VR" pad="P$1"/>
+<contactref element="D2" pad="C"/>
+<contactref element="PR2" pad="1"/>
+<wire x1="13.65" y1="33.93" x2="23.82" y2="41.71" width="0" layer="19" extent="1-1"/>
+<wire x1="35.6" y1="8.4" x2="13.65" y2="33.93" width="0" layer="19" extent="1-1"/>
+</signal>
+<signal name="N$4">
 <contactref element="D3" pad="C"/>
-<contactref element="VR" pad="P$1"/>
-<wire x1="23.82" y1="41.71" x2="28.55" y2="41.71" width="0" layer="19" extent="1-1"/>
-</signal>
-<signal name="N$2">
-<contactref element="R2" pad="2"/>
+<contactref element="C4" pad="1"/>
+<contactref element="D2" pad="A"/>
+<wire x1="13.65" y1="41.55" x2="28.55" y2="41.71" width="0" layer="19" extent="1-1"/>
+<wire x1="20.07" y1="28.35" x2="13.65" y2="41.55" width="0" layer="19" extent="1-1"/>
+</signal>
+<signal name="N$3">
+<contactref element="D3" pad="A"/>
+<contactref element="VR" pad="P$3"/>
+<contactref element="PR1" pad="1"/>
+<wire x1="27.6" y1="27.6" x2="28.55" y2="34.09" width="0" layer="19" extent="1-1"/>
+<wire x1="18.82" y1="41.71" x2="28.55" y2="34.09" width="0" layer="19" extent="1-1"/>
+</signal>
+<signal name="PR1">
+<contactref element="PR1" pad="2"/>
 <contactref element="J1" pad="1"/>
-<wire x1="27.6" y1="20.9" x2="27.6" y2="23.6" width="0.8128" layer="1"/>
-</signal>
-<signal name="N$3">
+<wire x1="27.6" y1="20.9" x2="27.6" y2="23.6" width="0" layer="19" extent="1-1"/>
+</signal>
+<signal name="PR2">
+<contactref element="PR2" pad="2"/>
 <contactref element="J1" pad="3"/>
-<contactref element="R1" pad="P$2"/>
-<wire x1="32.37" y1="23.47" x2="30.8" y2="21.9" width="0.8128" layer="1"/>
-<wire x1="30.8" y1="21.9" x2="30.8" y2="18.1" width="0.8128" layer="1"/>
-<wire x1="30.8" y1="18.1" x2="28.52" y2="15.82" width="0.8128" layer="1"/>
-<wire x1="28.52" y1="15.82" x2="27.6" y2="15.82" width="0.8128" layer="1"/>
+<wire x1="35.6" y1="4.4" x2="27.6" y2="15.82" width="0" layer="19" extent="1-1"/>
 </signal>
 </signals>

Commit message: added LOGO
Parts:
- added JP3: POWER_JACKPTH, SparkFun-Connectors:POWER_JACK_PTH
- added U$1: LOGO, SparkFun-Electromechanical:LOGO
- moved PR2 40.0 mm to (28.9, 45.8), turned to 90 degrees
- moved J1 28.3 mm to (18.8, 47.8), turned to 0 degrees
- moved PR1 24.5 mm to (13.7, 45.8), turned to 90 degrees
- moved D2 15.3 mm to (28.9, 37.9), turned to 90 degrees
- moved D3 14.9 mm to (13.7, 37.7), turned to 270 degrees
- moved R1 13.9 mm to (36.5, 41.8), turned to 0 degrees
- moved R3 12.7 mm to (29.3, 22.6), turned to 90 degrees
- moved R4 4.80 mm to (5.33, 32.2), turned to 90 degrees
- moved C2 2.50 mm to (17.6, 15.1), turned to 0 degrees
- moved LED1 2.44 mm to (5.31, 22.6)
- moved Q1 1.70 mm to (32.0, 33.4)
- moved D4 1.70 mm to (38.1, 34.5)
- moved T1 1.70 mm to (35.8, 17.6)
- moved D1 1.50 mm to (38.5, 16.3)
Connections:
- net GND: now also JP3.GND
- net VCC: now also JP3.PWR
Routing:
- net 555_DISCH: track 0.00 -> 51.8 mm
- net N$4: track 0.00 -> 22.5 mm
- net OUT: track 66.2 -> 47.1 mm, vias 1 -> 0
- net N$2: track 0.00 -> 7.78 mm
- net N$3: track 0.00 -> 7.56 mm
- net N$7: track 11.2 -> 5.18 mm
- net PR1: track 0.00 -> 5.10 mm
- net PR2: track 0.00 -> 5.02 mm
- net LOAD2-: track 11.6 -> 13.3 mm
- net LOAD1-: track 11.4 -> 13.0 mm
- net VCC: track 116.5 -> 115.0 mm
- net N$5: track 3.10 -> 4.58 mm
Other:
- board text removed: "Black"
- board text removed: "Red"
