File: eagle/555-dev-2.brd (EAGLE design)
At the start: 50 x 50 mm, 27 parts, among them IC1 NE555, Q1 IRF740, T1 2N2222

Commit message: ver 1
Parts:
- added U$1: LOGO, SparkFun-Electromechanical:LOGO
Other:
- board text removed: "Black"
- board text removed: "Red"
Changed lines of the file:
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@@
 <text x="42.9" y="23.9" size="1.9304" layer="21" font="vector" ratio="10" rot="R270">-
 +</text>
-<text x="23.1" y="7" size="1.27" layer="21" font="vector" ratio="10" rot="R180">Red</text>
-<text x="33.8" y="7" size="1.27" layer="21" font="vector" ratio="10" rot="R180">Black</text>
 </plain>
 <attributes>
@@
 <attribute name="PROD_ID" value="CONN-08197" x="12.9" y="-0.1" size="1.778" layer="27" display="off"/>
 </element>
+<element name="U$1" library="SparkFun-Electromechanical" package="LOGO" value="LOGO" x="28.8" y="6"/>
 </elements>
 <signals>
