File: eagle/555-dev-2.sch (EAGLE design)
At the start: 27 parts, among them IC1 NE555, Q1 IRF740, T1 2N2222

Commit message: ver 1
Parts:
- added U$1: LOGO, SparkFun-Electromechanical:LOGO
Changed lines of the file:
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@@
 <part name="P+2" library="supply1" deviceset="VCC" device=""/>
 <part name="GND3" library="supply1" deviceset="GND" device=""/>
+<part name="U$1" library="SparkFun-Electromechanical" deviceset="LOGO" device=""/>
 </parts>
 <sheets>
@@
 <instance part="P+2" gate="VCC" x="111.76" y="86.36"/>
 <instance part="GND3" gate="1" x="111.76" y="76.2"/>
+<instance part="U$1" gate="G$1" x="33.02" y="86.36"/>
 </instances>
 <busses>
